File: MAX31865_Layout_with_OLED.brd (EAGLE design)
At the start: 47.9 x 27 mm, 33 parts, among them IC1 MAX31865, IC2 MIC5225-3.3, IC3 ATMEGA328-AI, P1 LSP15, P2 LSP15, P3 LSP15, P4 LSP15, Q1 8/16/20MHz, X3 MINI-USB

Commit message: Add files via upload
Parts:
- added LED1: green, led:CHIPLED_0805
- added R3: 470, rcl1:R0603
Connections:
- new net N$14: LED1.A, R3.2
- net +5V: now also R3.1
- net GND: now also LED1.C
Routing:
- net GND: track 111.4 -> 117.1 mm, vias 7 -> 8
- net +5V: track 85.0 -> 89.6 mm
- net N$14: track 0.00 -> 1.59 mm
Changed lines of the file:
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@@
 </element>
 <element name="IC2" library="microbuilder" package="SOT23-5" value="MIC5225-3.3" x="13.17625" y="17.93875" smashed="yes" rot="R270">
-<attribute name="NAME" x="14.684375" y="14.757375" size="0.762" layer="25" ratio="10" rot="R90"/>
+<attribute name="NAME" x="10.795" y="17.05925" size="0.762" layer="25" ratio="10" rot="R90"/>
 <attribute name="VALUE" x="13.49375" y="14.439875" size="0.762" layer="27" ratio="10" rot="R90"/>
 </element>
@@
 <element name="U$2" library="microbuilder" package="MOUNTINGHOLE_2.5_PLATED" value="MOUNTINGHOLE2.5" x="11.5" y="3">
 <attribute name="BOM" value="EXCLUDE" x="11.5" y="3" size="1.778" layer="27" display="off"/>
+</element>
+<element name="LED1" library="led" package="CHIPLED_0805" value="green" x="41.195625" y="2.619375" smashed="yes" rot="R270">
+<attribute name="NAME" x="39.6875" y="0.873125" size="0.762" layer="25" ratio="10"/>
+<attribute name="VALUE" x="39.6875" y="2.301875" size="0.762" layer="27" ratio="10"/>
+</element>
+<element name="R3" library="rcl1" package="R0603" value="470" x="37.703125" y="2.619375" smashed="yes">
+<attribute name="NAME" x="36.433125" y="0.873125" size="0.762" layer="25" ratio="10"/>
+<attribute name="VALUE" x="36.67125" y="2.2225" size="0.762" layer="27" ratio="10"/>
 </element>
 </elements>
@@
 <wire x1="43.4975" y1="24.368125" x2="41.513125" y2="24.368125" width="0.508" layer="16"/>
 <wire x1="41.513125" y1="24.368125" x2="39.21125" y2="22.06625" width="0.508" layer="16"/>
+<contactref element="LED1" pad="C"/>
+<via x="43.100625" y="2.619375" extent="1-16" drill="0.6" diameter="1.4224" shape="octagon"/>
+<wire x1="43.100625" y1="2.619375" x2="41.75125" y2="2.619375" width="0.508" layer="16"/>
+<wire x1="41.75125" y1="2.619375" x2="39.290625" y2="5.08" width="0.508" layer="16"/>
+<wire x1="42.245625" y1="2.619375" x2="43.100625" y2="2.619375" width="0.508" layer="1"/>
 </signal>
 <signal name="VDD">
@@
 <wire x1="14.625" y1="12.94125" x2="13.890625" y2="13.675625" width="0.508" layer="1"/>
 <wire x1="32.0675" y1="8.5725" x2="33.81375" y2="6.82625" width="0.508" layer="1"/>
-<wire x1="34.55125" y1="6.19125" x2="34.44875" y2="6.19125" width="0.508" layer="1"/>
-<wire x1="34.44875" y1="6.19125" x2="33.81375" y2="6.82625" width="0.508" layer="1"/>
 <wire x1="20.811875" y1="10.54125" x2="20.0025" y2="11.350625" width="0.508" layer="1"/>
 <contactref element="P2" pad="P$1"/>
@@
 <wire x1="21.193125" y1="24.28875" x2="19.20875" y2="22.304375" width="0.508" layer="16"/>
 <wire x1="19.20875" y1="22.304375" x2="18.653125" y2="22.304375" width="0.508" layer="16"/>
+<contactref element="R3" pad="1"/>
+<wire x1="33.81375" y1="6.82625" x2="33.81375" y2="5.3975" width="0.508" layer="1"/>
+<wire x1="33.81375" y1="5.3975" x2="36.591875" y2="2.619375" width="0.508" layer="1"/>
+<wire x1="36.591875" y1="2.619375" x2="36.853125" y2="2.619375" width="0.508" layer="1"/>
+<wire x1="33.81375" y1="6.82625" x2="34.55125" y2="6.19125" width="0" layer="19" extent="1-16"/>
 </signal>
 <signal name="SDA">
@@
 <wire x1="8.5725" y1="5.3975" x2="8.5725" y2="0" width="0.1524" layer="1" style="shortdash"/>
 </signal>
+<signal name="N$14">
+<contactref element="R3" pad="2"/>
+<contactref element="LED1" pad="A"/>
+<wire x1="38.553125" y1="2.619375" x2="40.145625" y2="2.619375" width="0.508" layer="1"/>
+</signal>
 </signals>
