File: MAX31865_Layout_with_OLED.sch (EAGLE design)
At the start: 33 parts, among them IC1 MAX31865, IC2 MIC5225-3.3, IC3 ATMEGA328-AI, P1 LSP15, P2 LSP15, P3 LSP15, P4 LSP15, Q1 8/16/20MHz, X3 MINI-USB

Commit message: Add files via upload
Parts:
- added LED1: green, led:LEDCHIPLED_0805
- added R3: 470, rcl1:R-EU_R0603
Connections:
- new net N$14: LED1.A, R3.2
- net +5V: now also R3.1
- net GND: now also LED1.C
Changed lines of the file:
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@@
 <layer number="96" name="Values" color="7" fill="1" visible="yes" active="yes"/>
 <layer number="97" name="Info" color="7" fill="1" visible="yes" active="yes"/>
+<layer number="98" name="Guide" color="6" fill="1" visible="yes" active="yes"/>
 <layer number="99" name="SpiceOrder" color="7" fill="1" visible="no" active="no"/>
 <layer number="100" name="Muster" color="7" fill="1" visible="no" active="no"/>
@@
 <part name="U$19" library="microbuilder" deviceset="MOUNTINGHOLE" device="2.5"/>
 <part name="U$2" library="microbuilder" deviceset="MOUNTINGHOLE" device="2.5"/>
+<part name="LED1" library="led" deviceset="LED" device="CHIPLED_0805" value="green"/>
+<part name="SUPPLY5" library="supply2" deviceset="+5V" device="" value="+5V"/>
+<part name="R3" library="rcl1" deviceset="R-EU_" device="R0603" value="470"/>
+<part name="GND6" library="supply1" deviceset="GND" device=""/>
 </parts>
 <sheets>
@@
 <wire x1="40.64" y1="190.5" x2="40.64" y2="152.4" width="0.1524" layer="97" style="shortdash"/>
 <wire x1="10.16" y1="152.4" x2="40.64" y2="152.4" width="0.1524" layer="97" style="shortdash"/>
-<text x="106.68" y="137.16" size="2.54" layer="94" ratio="10">Max31865 Module</text>
+<text x="104.14" y="129.54" size="2.54" layer="94" ratio="10">Max31865 Module</text>
 <text x="205.74" y="30.48" size="2.54" layer="94" ratio="10">Arduino Mini-Pro</text>
 <text x="200.66" y="137.16" size="2.54" layer="94" ratio="10">OLED-Display I2C</text>
@@
 <attribute name="NAME" x="46.0375" y="174.6885" size="1.778" layer="95"/>
 </instance>
-<instance part="U$19" gate="G$1" x="142.24" y="170.18"/>
+<instance part="U$19" gate="G$1" x="152.4" y="157.48"/>
 <instance part="U$2" gate="G$1" x="152.4" y="170.18"/>
+<instance part="LED1" gate="G$1" x="132.08" y="162.56"/>
+<instance part="SUPPLY5" gate="+5V" x="132.08" y="177.8"/>
+<instance part="R3" gate="G$1" x="132.08" y="170.18" smashed="yes" rot="R270">
+<attribute name="NAME" x="135.6614" y="168.91" size="1.778" layer="95" ratio="10" rot="R90"/>
+<attribute name="VALUE" x="129.413" y="170.18" size="1.778" layer="96" ratio="10" rot="R270" align="center"/>
+</instance>
+<instance part="GND6" gate="1" x="132.08" y="154.94"/>
 </instances>
 <busses>
@@
 <pinref part="SUPPLY1" gate="+5V" pin="+5V"/>
 </segment>
+<segment>
+<pinref part="SUPPLY5" gate="+5V" pin="+5V"/>
+<pinref part="R3" gate="G$1" pin="1"/>
+</segment>
 </net>
 <net name="GND" class="0">
@@
 <pinref part="GND12" gate="1" pin="GND"/>
 </segment>
+<segment>
+<pinref part="LED1" gate="G$1" pin="C"/>
+<pinref part="GND6" gate="1" pin="GND"/>
+</segment>
 </net>
 <net name="SDA" class="0">
@@
 </segment>
 </net>
+<net name="N$14" class="0">
+<segment>
+<pinref part="R3" gate="G$1" pin="2"/>
+<pinref part="LED1" gate="G$1" pin="A"/>
+</segment>
+</net>
